File: schematics/nixie_clock.brd (EAGLE design)
At the start: 100 x 80 mm, 50 parts, among them IC1 LM7805, IC2 74141N, IC3 MEGA8-P, IC4 MAX1771-TH, IC5 DS1307-TH, Q1 IRF 830

Commit message: Updated Schematics
Parts:
- removed IC5: DS1307-TH, ds1307:DS1307
- added U$1: DS1307-TH, ds1307:DS1307
- moved G1 230.7 mm to (68.6, 24.1), turned to 180 degrees
- moved IC4 191.0 mm to (17.8, -12.7)
- moved NT4 156.1 mm to (-133.3, 68.6), turned to 180 degrees
- moved NT3 137.5 mm to (-149.9, 68.6), turned to 180 degrees
- moved D2 132.1 mm to (69.8, 49.5)
- moved NT2 125.1 mm to (-166.4, 68.6), turned to 180 degrees
- moved NT1 120.7 mm to (-182.9, 68.6), turned to 180 degrees
- moved C10 118.6 mm to (47.0, -26.7)
- moved IC1 113.0 mm to (10.2, -35.6)
- moved R1 112.1 mm to (64.8, 66.0)
- moved T9 99.1 mm to (-113.0, 45.7)
- moved L1 96.5 mm to (59.7, -3.81)
- moved C3 67.6 mm to (35.6, 92.7)
- moved IC3 64.1 mm to (-40.6, -33.0)
- moved IC2 44.6 mm to (-49.5, -11.4)
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Connections:
- net GND: now also U$1.4; no longer IC5.4
- net IC5: now also U$1.2; no longer IC5.2
- net N$25: now also U$1.8; no longer IC5.8
- net N$41: now also U$1.5; no longer IC5.5
- net N$42: now also U$1.6; no longer IC5.6
- net N$45: now also U$1.1; no longer IC5.1
- net N$47: now also U$1.3; no longer IC5.3
Other:
- board size 100 x 80 mm -> 202.9 x 129.5 mm
