File: schematics/nixie_clock.sch (EAGLE design)
At the start: 50 parts, among them IC1 LM7805, IC2 74141N, IC3 MEGA8-P, IC4 MAX1771-TH, IC5 DS1307-TH, Q1 IRF 830

Commit message: Updated Schematics
Parts:
- renumbered IC5 to U$1
Changed lines of the file:
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@@
 <?xml version="1.0" encoding="utf-8"?>
 <!DOCTYPE eagle SYSTEM "eagle.dtd">
-<eagle version="6.0">
+<eagle version="6.1">
 <drawing>
 <settings>
@@
 <part name="G1" library="battery" deviceset="CR2032H" device=""/>
 <part name="T9" library="transistor" deviceset="*-NPN-" device="TO92-CBE" technology="MPSA44"/>
-<part name="IC5" library="ds1307" deviceset="DS1307" device="-TH"/>
 <part name="IC4" library="max1771" deviceset="MAX1771" device="-TH"/>
 <part name="NT1" library="nixie" deviceset="NIXIE" device="-IN-12B"/>
@@
 <part name="NT3" library="nixie" deviceset="NIXIE" device="-IN-12B"/>
 <part name="NT4" library="nixie" deviceset="NIXIE" device="-IN-12B"/>
+<part name="U$1" library="ds1307" deviceset="DS1307" device="-TH"/>
 </parts>
 <sheets>
@@
 <instance part="G1" gate="1" x="-93.98" y="-40.64"/>
 <instance part="T9" gate="G$1" x="7.62" y="-22.86"/>
-<instance part="IC5" gate="G$1" x="-60.96" y="-38.1"/>
 <instance part="IC4" gate="MAX1771" x="33.02" y="2.54"/>
 <instance part="NT1" gate="G$1" x="-119.38" y="25.4"/>
@@
 <instance part="NT3" gate="G$1" x="-43.18" y="25.4"/>
 <instance part="NT4" gate="G$1" x="-5.08" y="25.4"/>
+<instance part="U$1" gate="G$1" x="-60.96" y="-38.1"/>
 </instances>
 <busses>
@@
 <wire x1="-93.98" y1="-53.34" x2="-93.98" y2="-55.88" width="0.1524" layer="91"/>
 <junction x="-93.98" y="-53.34"/>
-<pinref part="IC5" gate="G$1" pin="GND"/>
+<pinref part="U$1" gate="G$1" pin="GND"/>
 </segment>
 </net>
@@
 <wire x1="40.64" y1="-53.34" x2="30.48" y2="-53.34" width="0.1524" layer="91"/>
 <wire x1="30.48" y1="-53.34" x2="30.48" y2="-35.56" width="0.1524" layer="91"/>
-<pinref part="IC5" gate="G$1" pin="VCC"/>
 <wire x1="-45.72" y1="-30.48" x2="-33.02" y2="-30.48" width="0.1524" layer="91"/>
 <wire x1="30.48" y1="-35.56" x2="-33.02" y2="-35.56" width="0.1524" layer="91"/>
 <wire x1="-33.02" y1="-35.56" x2="-33.02" y2="-30.48" width="0.1524" layer="91"/>
+<pinref part="U$1" gate="G$1" pin="VCC"/>
 </segment>
 </net>
@@
 <wire x1="-43.18" y1="-53.34" x2="-43.18" y2="-45.72" width="0.1524" layer="91"/>
 <wire x1="-43.18" y1="-45.72" x2="-45.72" y2="-45.72" width="0.1524" layer="91"/>
-<pinref part="IC5" gate="G$1" pin="SDA"/>
+<pinref part="U$1" gate="G$1" pin="SDA"/>
 </segment>
 </net>
@@
 <wire x1="-40.64" y1="-55.88" x2="-40.64" y2="-40.64" width="0.1524" layer="91"/>
 <wire x1="-40.64" y1="-40.64" x2="-45.72" y2="-40.64" width="0.1524" layer="91"/>
-<pinref part="IC5" gate="G$1" pin="SCL"/>
+<pinref part="U$1" gate="G$1" pin="SCL"/>
 </segment>
 </net>
@@
 <pinref part="Q2" gate="G$1" pin="1"/>
 <wire x1="-78.74" y1="-38.1" x2="-83.82" y2="-38.1" width="0.1524" layer="91"/>
-<pinref part="IC5" gate="G$1" pin="XTAL2"/>
+<pinref part="U$1" gate="G$1" pin="XTAL2"/>
 </segment>
 </net>
@@
 <pinref part="Q2" gate="G$1" pin="2"/>
 <wire x1="-78.74" y1="-27.94" x2="-83.82" y2="-27.94" width="0.1524" layer="91"/>
-<pinref part="IC5" gate="G$1" pin="XTAL1"/>
+<pinref part="U$1" gate="G$1" pin="XTAL1"/>
 </segment>
 </net>
@@
 <pinref part="G1" gate="1" pin="+"/>
 <wire x1="-76.2" y1="-40.64" x2="-88.9" y2="-40.64" width="0.1524" layer="91"/>
-<pinref part="IC5" gate="G$1" pin="VBAT"/>
-</segment>
-</net>
+<pinref part="U$1" gate="G$1" pin="VBAT"/>
+</segment>
+</net>
